Commit message: add alexbotmini urdf&xml

File: alexbotmini_2(inuse)/urdf/alexbotmini.urdf (robot description, URDF)
Before this commit: robot alexbotmini, 13 links, 12 joints
Joints:
- joint leftjoint1: limit lower=-1 upper=1 effort=96 velocity=100 -> lower=-1 upper=1 effort=96 velocity=10.4719755
- joint leftjoint2: limit lower=-0.3 upper=0.2 effort=51 velocity=59 -> lower=-0.3 upper=0.2 effort=51 velocity=10.4719755
- joint leftjoint3: limit lower=-1 upper=1 effort=51 velocity=59 -> lower=-1 upper=1 effort=51 velocity=10.4719755
- joint leftjoint4: limit lower=-1 upper=1 effort=96 velocity=100 -> lower=-1 upper=1 effort=96 velocity=10.4719755
- joint leftjoint5: limit lower=-1 upper=1 effort=30 velocity=130 -> lower=-1 upper=1 effort=30 velocity=13.613568149999999
- joint leftjoint6: limit lower=-0.5 upper=0.5 effort=30 velocity=130 -> lower=-0.5 upper=0.5 effort=30 velocity=13.613568149999999
- joint rightjoint1: limit lower=-1 upper=1 effort=96 velocity=100 -> lower=-1 upper=1 effort=96 velocity=10.47
- joint rightjoint2: limit lower=-0.2 upper=0.3 effort=51 velocity=59 -> lower=-0.2 upper=0.3 effort=51 velocity=6.178465545
- joint rightjoint3: limit lower=-1 upper=1 effort=51 velocity=59 -> lower=-1 upper=1 effort=51 velocity=6.178465545
- joint rightjoint4: limit lower=-1 upper=1 effort=96 velocity=100 -> lower=-1 upper=1 effort=96 velocity=10.4719755
- joint rightjoint5: limit lower=-1 upper=1 effort=30 velocity=130 -> lower=-1 upper=1 effort=30 velocity=13.613568149999999
- joint rightjoint6: limit lower=-0.5 upper=0.5 effort=30 velocity=130 -> lower=-0.5 upper=0.5 effort=30 velocity=13.613568149999999
