Commit message: add pinocchio show
add pinocchio show

File: alexbotmini/urdf/alexbotmini_copy.urdf (robot description, URDF)
Before this commit: robot alexbotmini, 13 links, 12 joints
Links:
- link base_link: geometry collision box name=baselink size=0.16 0.16 0.12; visual mesh filename=/home/alexhuge/Documents/GitHub/Alexbotmini_urdf/alexbotmin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
- link leftlink1: geometry visual mesh filename=/home/alexhuge/Documents/GitHub/Alexbotmini_urdf/alexbotmin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
- link leftlink2: geometry collision box name=leftlink2 size=0.15 0.08 0.20; visual mesh filename=/home/alexhuge/Documents/GitHub/Alexbotmini_urdf/alexbotmin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
- link leftlink3: geometry collision cylinder length=0.1 name=leftlink3 radius=0.045; visual mesh filename=/home/alexhuge/Documents/GitHub/Alexbotmini_urdf/alexbotmin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
- link leftlink4: geometry collision box name=leftlink4 size=0.07 0.08 0.16; visual mesh filename=/home/alexhuge/Documents/GitHub/Alexbotmini_urdf/alexbotmin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
- link leftlink5: geometry visual mesh filename=/home/alexhuge/Documents/GitHub/Alexbotmini_urdf/alexbotmin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
- link leftlink6: geometry collision box size=0.1 0.24 0.01; visual mesh filename=/home/alexhuge/Documents/GitHub/Alexbotmini_urdf/alexbotmin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
- link rightlink1: geometry visual mesh filename=/home/alexhuge/Documents/GitHub/Alexbotmini_urdf/alexbotmin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
- link rightlink2: geometry collision box name=rightlink2 size=0.15 0.08 0.20; visual mesh filename=/home/alexhuge/Documents/GitHub/Alexbotmini_urdf/alexbotmin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
- link rightlink3: geometry collision cylinder length=0.1 name=rightlink3 radius=0.045; visual mesh filename=/home/alexhuge/Documents/GitHub/Alexbotmini_urdf/alexbotmin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
- link rightlink4: geometry collision box name=rightlink4 size=0.07 0.08 0.16; visual mesh filename=/home/alexhuge/Documents/GitHub/Alexbotmini_urdf/alexbotmin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
- link rightlink5: geometry visual mesh filename=/home/alexhuge/Documents/GitHub/Alexbotmini_urdf/alexbotmin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
- link rightlink6: geometry collision box size=0.1 0.24 0.01; visual mesh filename=/home/alexhuge/Documents/GitHub/Alexbotmini_urdf/alexbotmin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
